File: buttons/buttons.kicad_sch (KiCad schematic)
At the start: 49 parts, among them J1 Conn_01x04, SW1 SW_SPST, SW10 SW_SPST, SW11 SW_SPST, SW12 SW_SPST, SW13 SW_SPST, SW14 SW_SPST, SW15 SW_SPST, SW16 SW_SPST, SW2 SW_SPST, SW3 SW_SPST, SW4 SW_SPST, SW5 SW_SPST, SW6 SW_SPST, SW7 SW_SPST, SW8 SW_SPST, SW9 SW_SPST

Commit message: Added power LED
Parts:
- C1, C10, C11, C12, C13, C14, C15, C16, C2, C3, C4, C5, C6, C7, C8, C9: DPN (none) -> GMC10X5R106M10NT; MPN (none) -> 4713-GMC10X5R106M10NTCT-ND
Changed lines of the file:
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@@
       (effects (font (size 1.27 1.27)) hide)
     )
-    (property "DPN" "" (at 99.06 180.34 0)
-      (effects (font (size 1.27 1.27)) hide)
-    )
-    (property "MPN" "" (at 99.06 180.34 0)
+    (property "DPN" "GMC10X5R106M10NT" (at 99.06 180.34 0)
+      (effects (font (size 1.27 1.27)) hide)
+    )
+    (property "MPN" "4713-GMC10X5R106M10NTCT-ND" (at 99.06 180.34 0)
       (effects (font (size 1.27 1.27)) hide)
     )
@@
       (effects (font (size 1.27 1.27)) hide)
     )
-    (property "DPN" "" (at 109.22 180.34 0)
-      (effects (font (size 1.27 1.27)) hide)
-    )
-    (property "MPN" "" (at 109.22 180.34 0)
+    (property "DPN" "GMC10X5R106M10NT" (at 109.22 180.34 0)
+      (effects (font (size 1.27 1.27)) hide)
+    )
+    (property "MPN" "4713-GMC10X5R106M10NTCT-ND" (at 109.22 180.34 0)
       (effects (font (size 1.27 1.27)) hide)
     )
@@
       (effects (font (size 1.27 1.27)) hide)
     )
-    (property "DPN" "" (at 168.91 180.34 0)
-      (effects (font (size 1.27 1.27)) hide)
-    )
-    (property "MPN" "" (at 168.91 180.34 0)
+    (property "DPN" "GMC10X5R106M10NT" (at 168.91 180.34 0)
+      (effects (font (size 1.27 1.27)) hide)
+    )
+    (property "MPN" "4713-GMC10X5R106M10NTCT-ND" (at 168.91 180.34 0)
       (effects (font (size 1.27 1.27)) hide)
     )
@@
       (effects (font (size 1.27 1.27)) hide)
     )
-    (property "DPN" "" (at 68.58 180.34 0)
-      (effects (font (size 1.27 1.27)) hide)
-    )
-    (property "MPN" "" (at 68.58 180.34 0)
+    (property "DPN" "GMC10X5R106M10NT" (at 68.58 180.34 0)
+      (effects (font (size 1.27 1.27)) hide)
+    )
+    (property "MPN" "4713-GMC10X5R106M10NTCT-ND" (at 68.58 180.34 0)
       (effects (font (size 1.27 1.27)) hide)
     )
@@
       (effects (font (size 1.27 1.27)) hide)
     )
-    (property "DPN" "" (at 148.59 180.34 0)
-      (effects (font (size 1.27 1.27)) hide)
-    )
-    (property "MPN" "" (at 148.59 180.34 0)
+    (property "DPN" "GMC10X5R106M10NT" (at 148.59 180.34 0)
+      (effects (font (size 1.27 1.27)) hide)
+    )
+    (property "MPN" "4713-GMC10X5R106M10NTCT-ND" (at 148.59 180.34 0)
       (effects (font (size 1.27 1.27)) hide)
     )
@@
       (effects (font (size 1.27 1.27)) hide)
     )
-    (property "DPN" "" (at 158.75 180.34 0)
-      (effects (font (size 1.27 1.27)) hide)
-    )
-    (property "MPN" "" (at 158.75 180.34 0)
+    (property "DPN" "GMC10X5R106M10NT" (at 158.75 180.34 0)
+      (effects (font (size 1.27 1.27)) hide)
+    )
+    (property "MPN" "4713-GMC10X5R106M10NTCT-ND" (at 158.75 180.34 0)
       (effects (font (size 1.27 1.27)) hide)
     )
@@
       (effects (font (size 1.27 1.27)) hide)
     )
-    (property "DPN" "" (at 78.74 180.34 0)
-      (effects (font (size 1.27 1.27)) hide)
-    )
-    (property "MPN" "" (at 78.74 180.34 0)
+    (property "DPN" "GMC10X5R106M10NT" (at 78.74 180.34 0)
+      (effects (font (size 1.27 1.27)) hide)
+    )
+    (property "MPN" "4713-GMC10X5R106M10NTCT-ND" (at 78.74 180.34 0)
       (effects (font (size 1.27 1.27)) hide)
     )
@@
       (effects (font (size 1.27 1.27)) hide)
     )
-    (property "DPN" "" (at 38.1 180.34 0)
-      (effects (font (size 1.27 1.27)) hide)
-    )
-    (property "MPN" "" (at 38.1 180.34 0)
+    (property "DPN" "GMC10X5R106M10NT" (at 38.1 180.34 0)
+      (effects (font (size 1.27 1.27)) hide)
+    )
+    (property "MPN" "4713-GMC10X5R106M10NTCT-ND" (at 38.1 180.34 0)
       (effects (font (size 1.27 1.27)) hide)
     )
@@
       (effects (font (size 1.27 1.27)) hide)
     )
-    (property "DPN" "" (at 88.9 180.34 0)
-      (effects (font (size 1.27 1.27)) hide)
-    )
-    (property "MPN" "" (at 88.9 180.34 0)
+    (property "DPN" "GMC10X5R106M10NT" (at 88.9 180.34 0)
+      (effects (font (size 1.27 1.27)) hide)
+    )
+    (property "MPN" "4713-GMC10X5R106M10NTCT-ND" (at 88.9 180.34 0)
       (effects (font (size 1.27 1.27)) hide)
     )
@@
       (effects (font (size 1.27 1.27)) hide)
     )
-    (property "DPN" "" (at 129.54 180.34 0)
-      (effects (font (size 1.27 1.27)) hide)
-    )
-    (property "MPN" "" (at 129.54 180.34 0)
+    (property "DPN" "GMC10X5R106M10NT" (at 129.54 180.34 0)
+      (effects (font (size 1.27 1.27)) hide)
+    )
+    (property "MPN" "4713-GMC10X5R106M10NTCT-ND" (at 129.54 180.34 0)
       (effects (font (size 1.27 1.27)) hide)
     )
@@
       (effects (font (size 1.27 1.27)) hide)
     )
-    (property "DPN" "" (at 48.26 180.34 0)
-      (effects (font (size 1.27 1.27)) hide)
-    )
-    (property "MPN" "" (at 48.26 180.34 0)
+    (property "DPN" "GMC10X5R106M10NT" (at 48.26 180.34 0)
+      (effects (font (size 1.27 1.27)) hide)
+    )
+    (property "MPN" "4713-GMC10X5R106M10NTCT-ND" (at 48.26 180.34 0)
       (effects (font (size 1.27 1.27)) hide)
     )
@@
       (effects (font (size 1.27 1.27)) hide)
     )
-    (property "DPN" "" (at 119.38 180.34 0)
-      (effects (font (size 1.27 1.27)) hide)
-    )
-    (property "MPN" "" (at 119.38 180.34 0)
+    (property "DPN" "GMC10X5R106M10NT" (at 119.38 180.34 0)
+      (effects (font (size 1.27 1.27)) hide)
+    )
+    (property "MPN" "4713-GMC10X5R106M10NTCT-ND" (at 119.38 180.34 0)
       (effects (font (size 1.27 1.27)) hide)
     )
@@
       (effects (font (size 1.27 1.27)) hide)
     )
-    (property "DPN" "" (at 27.94 180.34 0)
-      (effects (font (size 1.27 1.27)) hide)
-    )
-    (property "MPN" "" (at 27.94 180.34 0)
+    (property "DPN" "GMC10X5R106M10NT" (at 27.94 180.34 0)
+      (effects (font (size 1.27 1.27)) hide)
+    )
+    (property "MPN" "4713-GMC10X5R106M10NTCT-ND" (at 27.94 180.34 0)
       (effects (font (size 1.27 1.27)) hide)
     )
@@
       (effects (font (size 1.27 1.27)) hide)
     )
-    (property "DPN" "" (at 58.42 180.34 0)
-      (effects (font (size 1.27 1.27)) hide)
-    )
-    (property "MPN" "" (at 58.42 180.34 0)
+    (property "DPN" "GMC10X5R106M10NT" (at 58.42 180.34 0)
+      (effects (font (size 1.27 1.27)) hide)
+    )
+    (property "MPN" "4713-GMC10X5R106M10NTCT-ND" (at 58.42 180.34 0)
       (effects (font (size 1.27 1.27)) hide)
     )
@@
       (effects (font (size 1.27 1.27)) hide)
     )
-    (property "DPN" "" (at 17.78 180.34 0)
-      (effects (font (size 1.27 1.27)) hide)
-    )
-    (property "MPN" "" (at 17.78 180.34 0)
+    (property "DPN" "GMC10X5R106M10NT" (at 17.78 180.34 0)
+      (effects (font (size 1.27 1.27)) hide)
+    )
+    (property "MPN" "4713-GMC10X5R106M10NTCT-ND" (at 17.78 180.34 0)
       (effects (font (size 1.27 1.27)) hide)
     )
@@
       (effects (font (size 1.27 1.27)) hide)
     )
-    (property "DPN" "" (at 138.43 180.34 0)
-      (effects (font (size 1.27 1.27)) hide)
-    )
-    (property "MPN" "" (at 138.43 180.34 0)
-      (effects (font (size 1.27 1.27)) hide)
-    )
+    (property "DPN" "GMC10X5R106M10NT" (at 138.43 180.34 0)
+      (effects (font (size 1.27 1.27)) hide)
+    )
+    (property "MPN" "4713-GMC10X5R106M10NTCT-ND" (at 138.43 180.34 0)
+      (effects (font (size 1.27 1.27)) hide)
+    )

Commit message: Picked components
Parts:
- J1: value Conn_01x04 -> DNP
Changed lines of the file:
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@@
       (effects (font (size 1.27 1.27)))
     )
-    (property "Value" "Conn_01x04" (at 175.26 143.51 0)
+    (property "Value" "DNP" (at 175.26 143.51 0)
       (effects (font (size 1.27 1.27)))
     )
